File: Modules/CVMod4/kicad/CVMod4_Panel.kicad_pcb (KiCad board)
At the start: 2 copper layers, 50.5 x 128.5 mm, 36 parts

Commit message: Add Interactive BOMs, resave all PCBs, move VU to THT.
Other:
- board text added: "CVMod4 v1.2"
- board text removed: "CVMod4 v1.0"
Changed lines of the file:
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@@
 	)
 	(paper "A4")
+	(title_block
+		(rev "v1.2")
+	)
 	(layers
 		(0 "F.Cu" signal)
@@
 		(layer "Edge.Cuts")
 	)
-	(gr_text "CVMod4 v1.0"
+	(gr_text "CVMod4 v1.2"
 		(at 64.008 40.005 0)
 		(layer "B.SilkS")
