File: Modules/CVMod8_V2/kicad/CVMod8_V2_Front.kicad_pcb (KiCad board)
At the start: 2 copper layers, 100.8 x 108.6 mm, 84 parts

Commit message: Add Interactive BOMs, resave all PCBs, move VU to THT.
Other:
- board text added: "CVMod8 V2 v2.1"
- board text removed: "CVMod8 V2 v2.0"
Changed lines of the file:
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@@
 	)
 	(paper "A4")
+	(title_block
+		(rev "v2.1")
+	)
 	(layers
 		(0 "F.Cu" signal)
@@
 		(layer "User.6")
 	)
-	(gr_text "CVMod8 V2 v2.0"
+	(gr_text "CVMod8 V2 v2.1"
 		(at 87.757 123.952 0)
 		(layer "B.SilkS")
