File: Modules/CVMod8_V2/kicad/CVMod8_V2.kicad_sch (KiCad schematic)
At the start: 138 parts, among them U1 TL074, U10 79L05, U2 TL074, U3 TL074, U4 TL074, U5 TL074, U6 TL074, U7 TL074, U8 TL074, U9 78L05

Commit message: Release SMD CVMod8 V2.
Parts:
- removed J_A1, J_A2, J_A3, J_A4, J_A5, J_A6, J_A7, J_A8: Conn_01x06_Male, Connector_PinHeader_2.54mm:PinHeader_1x06_P2.54mm_Vertical, symbol Connector:Conn_01x06_Male
- removed J_A11, J_A12, J_A13, J_A14: Conn_01x03_Male, Connector_PinHeader_2.54mm:PinHeader_1x03_P2.54mm_Vertical, symbol Connector:Conn_01x03_Male
- removed J_B1, J_B2, J_B3, J_B4, J_B5, J_B6, J_B7, J_B8: Conn_01x06_Female, Connector_PinHeader_2.54mm:PinHeader_1x06_P2.54mm_Vertical, symbol Connector:Conn_01x06_Female
- removed J_B11, J_B12, J_B13, J_B14: Conn_01x03_Female, Connector_PinHeader_2.54mm:PinHeader_1x03_P2.54mm_Vertical, symbol Connector:Conn_01x03_Female
- removed RN1, RN10, RN11, RN12, RN13, RN14, RN15, RN16, RN2, RN3, RN4, RN5, RN6, RN7, RN8, RN9: 100k, Resistor_THT:R_Array_SIP8, symbol Device:R_Pack04_SIP_Split
- added R10, R9: 1k, Resistor_SMD:R_0603_1608Metric_Pad0.98x0.95mm_HandSolder, symbol Device:R_Small
- added R19, R20, R21, R22, R23, R24, R25, R26, R27, R28, R29, R30, R31, R32, R33, R34, R35, R36, R37, R38, R39, R40, R41, R42, R43, R44, R45, R46, R47, R48, R49, R50, R51, R52, R53, R54, R55, R56, R57, R58, R59, R60, R61, R62, R63, R64, R65, R66, R67, R68, R69, R70, R71, R72, R73, R74, R75, R76, R77, R78, R79: 100k, Resistor_SMD:R_0603_1608Metric_Pad0.98x0.95mm_HandSolder, symbol Device:R_Small
- C1, C2: footprint Capacitor_THT:CP_Radial_D6.3mm_P2.50mm -> Capacitor_SMD:CP_Elec_6.3x5.3
- C10, C11, C12, C13, C14, C3, C4, C5, C6, C7, C8, C9: footprint Capacitor_THT:C_Disc_D7.0mm_W2.5mm_P5.00mm -> Capacitor_SMD:C_0603_1608Metric_Pad1.08x0.95mm_HandSolder
- D1, D2: value 1N4001 -> FM4001; footprint Diode_THT:D_DO-41_SOD81_P10.16mm_Horizontal -> Eurorack:D_SOD-123F_AH
- R1, R11, R12, R13, R14, R15, R16, R2, R3, R4, R5, R6, R7, R8: footprint Resistor_THT:R_Axial_DIN0207_L6.3mm_D2.5mm_P10.16mm_Horizontal -> Resistor_SMD:R_0603_1608Metric_Pad0.98x0.95mm_HandSolder
- R17, R18: value 1k -> 100k; footprint Resistor_THT:R_Axial_DIN0207_L6.3mm_D2.5mm_P10.16mm_Horizontal -> Resistor_SMD:R_0603_1608Metric_Pad0.98x0.95mm_HandSolder
- U1, U2, U3, U4, U5, U6, U7, U8: footprint Package_DIP:DIP-14_W7.62mm_Socket_LongPads -> Eurorack:SO-14_3.9x8.65mm_P1.27mm_AH
- U10, U9: footprint Package_TO_SOT_THT:TO-92_Inline_Wide -> Package_TO_SOT_SMD:SOT-89-3_Handsoldering
Connections:
- net +12V: now also C11.2, C13.2; no longer C10.2, C8.2
- net +5V: now also C4.1; no longer C5.1
- net -12V: now also C10.1, C5.2, C8.1; no longer C11.1, C13.1, C4.2
- net FWD1: now also R30.1
- net FWD2: now also R38.1
- net FWD3: now also R46.1
- net FWD4: now also R54.1
- net FWD5: now also R62.1
- net FWD6: now also R70.1
- net FWD7: now also R78.1
- net GND: now also C10.2, C11.1, C13.1, C4.2, C5.1, C8.2; no longer C10.1, C11.2, C13.2, C4.1, C5.2, C8.1
- net LED1: now also LD1.2 (A), R9.2; no longer R1.2
- net LED2: now also LD2.2 (A), R10.2; no longer R2.2
- net LED3: now also LD3.2 (A), R11.2; no longer R3.2
- net LED4: now also LD4.2 (A), R12.2; no longer R4.2
- net LED5: now also LD5.2 (A), R13.2; no longer R5.2
- net LED6: now also LD6.2 (A), R14.2; no longer R6.2
- net LED7: now also LD7.2 (A), R15.2; no longer R7.2
- net LED8: now also LD8.2 (A), R16.2; no longer R8.2
- net OFS1: now also P_OFS1.2
- net OFS2: now also P_OFS2.2
- net OFS3: now also P_OFS3.2
- net OFS4: now also P_OFS4.2
- net OFS5: now also P_OFS5.2
- net OFS6: now also P_OFS6.2
- net OFS7: now also P_OFS7.2
- net OFS8: now also P_OFS8.2
- net OUT1: now also R1.1, SW_FWD1.1 (A), R19.2
- net OUT2: now also R2.1, SW_FWD2.1 (A), R26.2
- net OUT3: now also R3.1, SW_FWD3.1 (A), R34.2
- net OUT4: now also R4.1, SW_FWD4.1 (A), R42.2
- net OUT5: now also R5.1, SW_FWD5.1 (A), R50.2
- net OUT6: now also R6.1, SW_FWD6.1 (A), R58.2
- net OUT7: now also R7.1, SW_FWD7.1 (A), R66.2
- net OUT8: now also R8.1, R74.2
- net at P_ATN2.2: now also U2.3 (+)
- net at J_IN2.SIG, P_ATN2.3: now also R25.1
- net at J_OUT5.SIG: now also R5.2; no longer R15.2
- net at U7.9 (-): now also R67.2, R68.2, R70.2, R71.1
- net at R11.1: now also U3.8, R37.1, R39.2; no longer SW_FWD1.1 (A)
- net at J_OUT1.SIG: now also R1.2; no longer R11.2
- net at P_ATN3.2: now also U3.3 (+)
- net at J_IN3.SIG, P_ATN3.3: now also R33.1
- net at U4.13 (-): now also R42.1, R45.2
- net at U7.8: now also R15.1, R69.1, R71.2; no longer R7.1
- net at U2.8: now also R10.1, R29.1, R31.2; no longer R2.1
- net at U2.13 (-): now also R26.1, R29.2
- net at R12.1: now also U4.8, R45.1, R47.2; no longer SW_FWD2.1 (A)
- net at U6.9 (-): now also R59.2, R60.2, R62.2, R63.1
- net at U6.6 (-), U6.7: now also R60.1
- net at R13.1: now also U5.8, R53.1, R55.2; no longer SW_FWD3.1 (A)
- net at U4.2 (-): now also R40.1, R41.2
- net at U4.1: now also R40.2, R43.1
- net at U8.8: now also R16.1, R77.1, R79.2; no longer R8.1
- net at U3.13 (-): now also R34.1, R37.2
- net at U8.3 (+): now also P_ATN8.2
- net at R18.1: now also J_IN1.SIG, P_ATN1.3
- net at J_IN8.SIG, P_ATN8.3: now also R73.1
- net at R14.1: now also U6.8, R61.1, R63.2; no longer SW_FWD4.1 (A)
- net at P_ATN4.2: now also U4.3 (+)
- net at J_IN4.SIG, P_ATN4.3: now also R41.1
- net at U1.6 (-), U1.7: now also R21.1
- net at U5.2 (-): now also R48.1, R49.2
- net at J_OUT3.SIG: now also R3.2; no longer R13.2
- net at U7.13 (-): now also R66.1, R69.2
- net at R17.1: now also R18.2, U1.2 (-); no longer SW_FWD7.1 (A)
- net at P_ATN7.2: now also U7.3 (+)
- net at J_IN7.SIG, P_ATN7.3: now also R65.1
- net at U8.9 (-): now also R75.2, R76.2, R78.2, R79.1
- net at U3.9 (-): now also R35.2, R36.2, R38.2, R39.1
- net at U3.6 (-), U3.7: now also R36.1
- net at U7.6 (-), U7.7: now also R68.1
- net at J_OUT4.SIG: now also R4.2; no longer R14.2
- net at U6.13 (-): now also R58.1, R61.2
- net at U4.6 (-), U4.7: now also R44.1
- net at U1.8: now also R22.1, R23.2, R9.1; no longer R1.1
- net at U2.1: now also R24.2, R27.1
- net at U2.9 (-): now also R27.2, R28.2, R30.2, R31.1
- net at U5.1: now also R48.2, R51.1
- net at U5.3 (+): now also P_ATN5.2
- net at U8.1: now also R72.2, R75.1
- net at U5.9 (-): now also R51.2, R52.2, R54.2, R55.1
- net at U1.9 (-): now also R20.2, R21.2, R23.1
- net at U8.2 (-): now also R72.1, R73.2
- net at U1.13 (-): now also R19.1, R22.2
- net at U6.1: now also R56.2, R59.1
- net at U6.2 (-): now also R56.1, R57.2
- net at U6.3 (+): now also P_ATN6.2
- net at U5.6 (-), U5.7: now also R52.1
- net at U7.2 (-): now also R64.1, R65.2
- net at U7.1: now also R64.2, R67.1
- net at J_IN6.SIG, P_ATN6.3: now also R57.1
- net at U5.13 (-): now also R50.1, R53.2
- net at U4.9 (-): now also R43.2, R44.2, R46.2, R47.1
- net at J_IN5.SIG, P_ATN5.3: now also R49.1
- net at U1.3 (+): now also P_ATN1.2
- net at J_OUT6.SIG: now also R6.2; no longer R16.2
- net at U3.1: now also R32.2, R35.1
- net at U3.2 (-): now also R32.1, R33.2
- net at U8.6 (-), U8.7: now also R76.1
- net at U8.13 (-): now also R74.1, R77.2
- net at J_OUT8.SIG: now also R8.2; no longer R18.2
- net at U2.2 (-): now also R24.1, R25.2
- net at U1.1: now also R17.2, R20.1
- net at J_OUT2.SIG: now also R2.2; no longer R12.2
- net at J_OUT7.SIG: now also R7.2; no longer R17.2
- net at U2.6 (-), U2.7: now also R28.1
- no-connect marks 25 -> 23
