File: Modules/CVMod8_V2/kicad/CVMod8_V2_Panel.kicad_pcb (KiCad board)
At the start: 2 copper layers, 101.3 x 128.5 mm, 66 parts

Commit message: Add Interactive BOMs, resave all PCBs, move VU to THT.
Other:
- board text added: "CVMod8 V2 v2.1"
- board text removed: "CVMod8 V2 v2.0"
Changed lines of the file:
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@@
 	)
 	(paper "A4")
+	(title_block
+		(rev "v2.1")
+	)
 	(layers
 		(0 "F.Cu" signal)
@@
 		(layer "Edge.Cuts")
 	)
-	(gr_text "CVMod8 V2 v2.0"
+	(gr_text "CVMod8 V2 v2.1"
 		(at 87.884 40.005 0)
 		(layer "B.SilkS")

Commit message: Release SMD CVMod8 V2.
Other:
- board text added: "CVMod8 V2 v2.2"
- board text removed: "CVMod8 V2 v2.1"
Changed lines of the file:
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@@
 	(paper "A4")
 	(title_block
-		(rev "v2.1")
+		(rev "v2.2")
 	)
 	(layers
@@
 		(layer "Edge.Cuts")
 	)
-	(gr_text "CVMod8 V2 v2.1"
+	(gr_text "CVMod8 V2 v2.2\n"
 		(at 87.884 40.005 0)
 		(layer "B.SilkS")
