File: Modules/KickAid/kicad/KickAid_Front.kicad_pcb (KiCad board)
At the start: 2 copper layers, 39.8 x 108.6 mm, 52 parts, among them U7 LM358

Commit message: Update KickAid PCBs.
Connections:
- J_IN pad SW: unconnected-(J_IN1-PadSW) -> GND
Other:
- board text added: "KickAid v1.2"
- board text removed: "KickAid v1.0"
Changed lines of the file:
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@@
 	(net 52 "unconnected-(J_RET1-PadSW)")
 	(net 53 "unconnected-(J_OUT1-PadSW)")
-	(net 54 "unconnected-(J_IN1-PadSW)")
-	(net 55 "unconnected-(J_GATE1-PadSW)")
-	(net 56 "Net-(J_B2-Pin_6)")
-	(net 57 "unconnected-(J_ENV1-PadSW)")
-	(net 58 "Net-(D7-K)")
-	(net 59 "Net-(D11-A)")
-	(net 60 "Net-(RN1A-R1.1)")
+	(net 54 "unconnected-(J_GATE1-PadSW)")
+	(net 55 "Net-(J_B2-Pin_6)")
+	(net 56 "unconnected-(J_ENV1-PadSW)")
+	(net 57 "Net-(D7-K)")
+	(net 58 "Net-(D11-A)")
+	(net 59 "Net-(RN1A-R1.1)")
 	(footprint "LED_THT:LED_D3.0mm_FlatTop"
 		(layer "F.Cu")
@@
 			(layers "*.Cu" "*.Mask")
 			(remove_unused_layers no)
-			(net 56 "Net-(J_B2-Pin_6)")
+			(net 55 "Net-(J_B2-Pin_6)")
 			(pintype "passive")
 		)
@@
 		(tags "LED Round FlatTop diameter 3.0mm 2 pins")
 		(property "Reference" "LD_K"
-			(at 4.323 0 -90)
+			(at 4.323 0 270)
 			(layer "F.SilkS")
 			(effects
@@
 			(layers "*.Cu" "*.Mask")
 			(remove_unused_layers no)
-			(net 55 "unconnected-(J_GATE1-PadSW)")
+			(net 54 "unconnected-(J_GATE1-PadSW)")
 			(pintype "passive+no_connect")
 		)
@@
 			(layers "*.Cu" "*.Mask")
 			(remove_unused_layers no)
-			(net 57 "unconnected-(J_ENV1-PadSW)")
+			(net 56 "unconnected-(J_ENV1-PadSW)")
 			(pintype "passive+no_connect")
 		)
@@
 			(layers "*.Cu" "*.Mask")
 			(remove_unused_layers no)
-			(net 54 "unconnected-(J_IN1-PadSW)")
-			(pintype "passive+no_connect")
+			(net 1 "GND")
+			(pintype "passive")
 		)
 		(zone
@@
 			(layers "*.Cu" "*.Mask")
 			(remove_unused_layers no)
-			(net 60 "Net-(RN1A-R1.1)")
+			(net 59 "Net-(RN1A-R1.1)")
 			(pintype "passive")
 		)
@@
 			(layers "*.Cu" "*.Mask")
 			(remove_unused_layers no)
-			(net 59 "Net-(D11-A)")
+			(net 58 "Net-(D11-A)")
 			(pinfunction "Pin_3")
 			(pintype "passive")
@@
 			(layers "*.Cu" "*.Mask")
 			(remove_unused_layers no)
-			(net 58 "Net-(D7-K)")
+			(net 57 "Net-(D7-K)")
 			(pinfunction "Pin_2")
 			(pintype "passive")
@@
 			(layers "*.Cu" "*.Mask")
 			(remove_unused_layers no)
-			(net 59 "Net-(D11-A)")
+			(net 58 "Net-(D11-A)")
 			(pinfunction "A")
 			(pintype "passive")
@@
 			(layers "*.Cu" "*.Mask")
 			(remove_unused_layers no)
-			(net 59 "Net-(D11-A)")
+			(net 58 "Net-(D11-A)")
 			(pinfunction "K")
 			(pintype "passive")
@@
 			(layers "*.Cu" "*.Mask")
 			(remove_unused_layers no)
-			(net 58 "Net-(D7-K)")
+			(net 57 "Net-(D7-K)")
 			(pinfunction "A")
 			(pintype "passive")
@@
 			(layers "*.Cu" "*.Mask")
 			(remove_unused_layers no)
-			(net 60 "Net-(RN1A-R1.1)")
+			(net 59 "Net-(RN1A-R1.1)")
 			(pinfunction "R1.1")
 			(pintype "passive")
@@
 			(layers "*.Cu" "*.Mask")
 			(remove_unused_layers no)
-			(net 56 "Net-(J_B2-Pin_6)")
+			(net 55 "Net-(J_B2-Pin_6)")
 			(pinfunction "Pin_6")
 			(pintype "passive")
@@
 			(layers "*.Cu" "*.Mask")
 			(remove_unused_layers no)
-			(net 58 "Net-(D7-K)")
+			(net 57 "Net-(D7-K)")
 			(pinfunction "K")
 			(pintype "passive")
@@
 		(layer "Edge.Cuts")
 	)
-	(gr_text "KickAid v1.0"
+	(gr_text "KickAid v1.2"
 		(at 63.5 129.794 0)
 		(layer "B.SilkS")
@@
 		(width 0.25)
 		(layer "B.Cu")
-		(net 56)
+		(net 55)
 	)
 	(segment
@@
 		(width 0.25)
 		(layer "B.Cu")
-		(net 56)
+		(net 55)
 	)
 	(segment
@@
 		(width 0.25)
 		(layer "B.Cu")
-		(net 56)
+		(net 55)
 	)
 	(segment
@@
 		(width 0.25)
 		(layer "B.Cu")
-		(net 56)
+		(net 55)
 	)
 	(segment
@@
 		(width 0.25)
 		(layer "F.Cu")
-		(net 58)
+		(net 57)
 	)
 	(segment
@@
 		(width 0.25)
 		(layer "F.Cu")
-		(net 58)
+		(net 57)
 	)
 	(segment
@@
 		(width 0.25)
 		(layer "F.Cu")
-		(net 58)
+		(net 57)
 	)
 	(segment
@@
 		(width 0.25)
 		(layer "F.Cu")
-		(net 59)
+		(net 58)
 	)
 	(segment
@@
 		(width 0.25)
 		(layer "F.Cu")
-		(net 59)
+		(net 58)
 	)
 	(segment
@@
 		(width 0.25)
 		(layer "F.Cu")
-		(net 59)
+		(net 58)
 	)
 	(segment
@@
 		(width 0.25)
 		(layer "F.Cu")
-		(net 59)
+		(net 58)
 	)
 	(segment
@@
 		(width 0.25)
 		(layer "F.Cu")
-		(net 59)
+		(net 58)
 	)
 	(segment
@@
 		(width 0.25)
 		(layer "F.Cu")
-		(net 59)
+		(net 58)
 	)
 	(segment
@@
 		(width 0.25)
 		(layer "F.Cu")
-		(net 59)
+		(net 58)
 	)
 	(segment
@@
 		(width 0.25)
 		(layer "F.Cu")
-		(net 59)
+		(net 58)
 	)
 	(via
@@
 		(drill 0.3)
 		(layers "F.Cu" "B.Cu")
-		(net 59)
+		(net 58)
 	)
 	(segment
@@
 		(width 0.25)
 		(layer "B.Cu")
-		(net 59)
+		(net 58)
 	)
 	(segment
@@
 		(width 0.25)
 		(layer "B.Cu")
-		(net 59)
+		(net 58)
 	)
 	(segment
@@
 		(width 0.25)
 		(layer "B.Cu")
-		(net 59)
+		(net 58)
 	)
 	(segment
@@
 		(width 0.25)
 		(layer "B.Cu")
-		(net 60)
+		(net 59)
 	)
 	(segment
@@
 		(width 0.25)
 		(layer "B.Cu")
-		(net 60)
+		(net 59)
 	)
 	(zone
