File: Modules/KickAid/kicad/KickAid_Main.kicad_pcb (KiCad board)
At the start: 2 copper layers, 39.8 x 108.6 mm, 79 parts, among them Q1 BCM847BS, U1 TL074, U2 TL074, U3 TL074, U4 TL074, U5 TL074, U6 LM324, U8 74HC04, U9 78L05

Commit message: Update KickAid PCBs.
Parts:
- C22: value 100pF -> 47pF
- R10: value 10k -> 15k
- R27: value 160k -> 120k
Other:
- board text added: "KickAid v1.2"
- board text removed: "KickAid v1.1"
Changed lines of the file:
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@@
 			)
 		)
-		(property "Value" "10k"
+		(property "Value" "15k"
 			(at 1.27 -2.37 0)
 			(layer "B.Fab")
@@
 			)
 		)
-		(property "Value" "100pF"
+		(property "Value" "47pF"
 			(at 2.5 -2.5 0)
 			(layer "B.Fab")
@@
 			)
 		)
-		(property "Value" "160k"
+		(property "Value" "120k"
 			(at 1.27 -2.37 0)
 			(layer "B.Fab")
@@
 			(layer "B.SilkS")
 		)
-		(fp_text user "RED"
-			(at -2.032 -4.318 90)
-			(unlocked yes)
+		(fp_text user "PWR"
+			(at -2.032 -2.032 -90)
 			(layer "B.SilkS")
 			(effects
@@
 					(thickness 0.15)
 				)
-				(justify left mirror)
+				(justify mirror)
 			)
 		)
-		(fp_text user "PWR"
-			(at -2.032 -2.032 -90)
+		(fp_text user "RED"
+			(at -2.032 -4.318 90)
+			(unlocked yes)
 			(layer "B.SilkS")
 			(effects
@@
 					(thickness 0.15)
 				)
-				(justify mirror)
+				(justify left mirror)
 			)
 		)
 		(pad "1" thru_hole circle
 			(at 0 5.08 180)
-			(size 1.524 1.524)
-			(drill 0.762)
+			(size 1.7 1.7)
+			(drill 1)
 			(layers "*.Cu" "*.Mask")
 			(remove_unused_layers no)
@@
 		(pad "1" thru_hole circle
 			(at 2.54 5.08 180)
-			(size 1.524 1.524)
-			(drill 0.762)
+			(size 1.7 1.7)
+			(drill 1)
 			(layers "*.Cu" "*.Mask")
 			(remove_unused_layers no)
@@
 		(pad "2" thru_hole circle
 			(at 0 -2.54 180)
-			(size 1.524 1.524)
-			(drill 0.762)
+			(size 1.7 1.7)
+			(drill 1)
 			(layers "*.Cu" "*.Mask")
 			(remove_unused_layers no)
@@
 		(pad "2" thru_hole circle
 			(at 0 0 180)
-			(size 1.524 1.524)
-			(drill 0.762)
+			(size 1.7 1.7)
+			(drill 1)
 			(layers "*.Cu" "*.Mask")
 			(remove_unused_layers no)
@@
 		(pad "2" thru_hole circle
 			(at 0 2.54 180)
-			(size 1.524 1.524)
-			(drill 0.762)
+			(size 1.7 1.7)
+			(drill 1)
 			(layers "*.Cu" "*.Mask")
 			(remove_unused_layers no)
@@
 		(pad "2" thru_hole circle
 			(at 2.54 -2.54 180)
-			(size 1.524 1.524)
-			(drill 0.762)
+			(size 1.7 1.7)
+			(drill 1)
 			(layers "*.Cu" "*.Mask")
 			(remove_unused_layers no)
@@
 		(pad "2" thru_hole circle
 			(at 2.54 0 180)
-			(size 1.524 1.524)
-			(drill 0.762)
+			(size 1.7 1.7)
+			(drill 1)
 			(layers "*.Cu" "*.Mask")
 			(remove_unused_layers no)
@@
 		(pad "2" thru_hole circle
 			(at 2.54 2.54 180)
-			(size 1.524 1.524)
-			(drill 0.762)
+			(size 1.7 1.7)
+			(drill 1)
 			(layers "*.Cu" "*.Mask")
 			(remove_unused_layers no)
@@
 		(pad "3" thru_hole rect
 			(at 0 -5.08 180)
-			(size 1.524 1.524)
-			(drill 0.762)
+			(size 1.7 1.7)
+			(drill 1)
 			(layers "*.Cu" "*.Mask")
 			(remove_unused_layers no)
@@
 		(pad "3" thru_hole rect
 			(at 2.54 -5.08 180)
-			(size 1.524 1.524)
-			(drill 0.762)
+			(size 1.7 1.7)
+			(drill 1)
 			(layers "*.Cu" "*.Mask")
 			(remove_unused_layers no)
@@
 		(layer "Edge.Cuts")
 	)
-	(gr_text "KickAid v1.1"
+	(gr_text "KickAid v1.2\n"
 		(at 45.466 98.552 270)
 		(layer "B.SilkS")

Commit message: Add Interactive BOMs, resave all PCBs, move VU to THT.
Parts:
- R34: value 100k -> 240k
Changed lines of the file:
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@@
 	)
 	(paper "A4")
+	(title_block
+		(rev "v1.2")
+	)
 	(layers
 		(0 "F.Cu" signal)
@@
 			)
 		)
-		(property "Value" "100k"
+		(property "Value" "240k"
 			(at 1.27 -2.37 180)
 			(layer "B.Fab")
