File: Modules/KickAid/kicad/KickAid_Panel.kicad_pcb (KiCad board)
At the start: 2 copper layers, 40.3 x 128.5 mm, 30 parts

Commit message: Update KickAid PCBs.
Other:
- board text added: "KickAid v1.2"
- board text removed: "KickAid v1.0"
Changed lines of the file:
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@@
 		(layer "Edge.Cuts")
 	)
-	(gr_text "KickAid v1.0"
+	(gr_text "KickAid v1.2"
 		(at 81.915 69.85 90)
 		(layer "B.SilkS")
