File: Modules/Nucleus/kicad/Nucleus_Main.kicad_pcb (KiCad board)
At the start: 2 copper layers, 39.8 x 55.5 mm, 26 parts, among them U1 LM358, U4 74HC04, U5 78L05

Commit message: Upgrade Nucleus to 1.2, fix triggers not working.
Parts:
- R1: value 220 -> 10
