File: Modules/R&F/kicad/R&F_Panel.kicad_pcb (KiCad board)
At the start: 2 copper layers, 15 x 128.5 mm, 14 parts

Commit message: Add Interactive BOMs, resave all PCBs, move VU to THT.
Other:
- board text added: "R&F v1.1"
- board text removed: "R&F v1.0"
