File: Modules/S&S/kicad/S&S_Back.kicad_pcb (KiCad board)
At the start: 2 copper layers, 14.5 x 97.6 mm, 26 parts, among them Q2 J112, U1 TL074

Commit message: Add Interactive BOMs, resave all PCBs, move VU to THT.
Parts:
- C11: value 10uF (Film) -> 2.2uF (Film)
