File: Modules/VU/kicad/VU_Panel.kicad_pcb (KiCad board)
At the start: 2 copper layers, 9.8 x 128.5 mm, 18 parts

Commit message: Add Interactive BOMs, resave all PCBs, move VU to THT.
Other:
- board text added: "VU v1.1"
- board text removed: "VU v1.0"
Changed lines of the file:
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@@
 	)
 	(paper "A4")
+	(title_block
+		(rev "v1.1")
+	)
 	(layers
 		(0 "F.Cu" signal)
@@
 		(layer "Edge.Cuts")
 	)
-	(gr_text "VU v1.0"
+	(gr_text "VU v1.1"
 		(at 92.075 74.93 90)
 		(layer "B.SilkS")
