File: Modules/VU/kicad/VU_THT.kicad_sch (KiCad schematic)
At the start: 65 parts, among them U1 LM3914N, U2 TL074, U3 TL074, U4 78L05

Commit message: Update label on VU THT schematic.
Other:
- title: Avalon Harmonics VU -> Avalon Harmonics VU (THT)
