File: Modules/iVCA/kicad/iVCA_Front.kicad_pcb (KiCad board)
At the start: 2 copper layers, 19.5 x 108.6 mm, 21 parts

Commit message: Add Interactive BOMs, resave all PCBs, move VU to THT.
Parts:
- removed the G*** at (69.2, 65.8)
- gave numbers to parts that had none: 1
Other:
- board text added: "iVCA v1.4"
- board text removed: "iVCA v1.0"
