File: Modules/iVCA/kicad/iVCA_Panel.kicad_pcb (KiCad board)
At the start: 2 copper layers, 20 x 128.5 mm, 14 parts

Commit message: Add Interactive BOMs, resave all PCBs, move VU to THT.
Parts:
- removed the G*** at (69.1, 59.3)
Other:
- board text added: "iVCA v1.4"
- board text removed: "iVCA v1.0"
